File: Electronics/PCB/GSP-1.0/GSP-1.0.kicad_sch (KiCad schematic)
At the start: 46 parts, among them J1 USB_C_Receptacle_USB2.0, Q1 ASS8050-L-HF, Q2 ASS8050-L-HF, SW1 SW_Push, SW2 SW_Push, SW3 SW_Push, SW4 SW_Push, SW5 SW_Push, SW6 SW_Push, SW7 SW_Push, SW8 SW_Push, U1 ESP32-S2-WROOM-I, U2 128x64_2.42"_OLED, U3 AZ1117-3.3, U4 AZ1117-3.3

Commit message: Final 1.0 version with PCB ordered
Parts:
- added C4, C5: 10uF, Capacitor_SMD:C_0805_2012Metric_Pad1.18x1.45mm_HandSolder, symbol Device:C
Connections:
- net +5V: now also C5.1
- net GNDREF: now also C4.1, C5.2
- net at BT1.1 (+), U3.3 (VI): now also C4.2
Changed lines of the file:
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@@
   (junction (at 104.14 50.8) (diameter 0) (color 0 0 0 0)
   )
+  (junction (at 41.91 55.88) (diameter 0) (color 0 0 0 0)
+  )
   (junction (at 104.14 43.18) (diameter 0) (color 0 0 0 0)
   )
@@
   (junction (at 351.79 160.02) (diameter 0) (color 0 0 0 0)
   )
+  (junction (at 69.85 58.42) (diameter 0) (color 0 0 0 0)
+  )
   (junction (at 162.56 120.65) (diameter 0) (color 0 0 0 0)
   )
@@
     (stroke (width 0) (type default) (color 0 0 0 0))
   )
+  (wire (pts (xy 69.85 58.42) (xy 72.39 58.42))
+    (stroke (width 0) (type default) (color 0 0 0 0))
+  )
   (wire (pts (xy 227.33 173.99) (xy 229.87 173.99))
     (stroke (width 0) (type default) (color 0 0 0 0))
@@
     (stroke (width 0) (type default) (color 0 0 0 0))
   )
-  (wire (pts (xy 69.85 59.69) (xy 69.85 57.15))
+  (wire (pts (xy 69.85 59.69) (xy 69.85 58.42))
     (stroke (width 0) (type default) (color 0 0 0 0))
   )
@@
     (stroke (width 0) (type default) (color 0 0 0 0))
   )
-  (wire (pts (xy 41.91 54.61) (xy 41.91 57.15))
+  (wire (pts (xy 41.91 54.61) (xy 41.91 55.88))
     (stroke (width 0) (type default) (color 0 0 0 0))
   )
@@
     (stroke (width 0) (type default) (color 0 0 0 0))
   )
+  (wire (pts (xy 35.56 55.88) (xy 41.91 55.88))
+    (stroke (width 0) (type default) (color 0 0 0 0))
+  )
   (wire (pts (xy 69.85 203.2) (xy 34.29 203.2))
     (stroke (width 0) (type default) (color 0 0 0 0))
@@
     (stroke (width 0) (type default) (color 0 0 0 0))
   )
+  (wire (pts (xy 41.91 55.88) (xy 41.91 57.15))
+    (stroke (width 0) (type default) (color 0 0 0 0))
+  )
   (wire (pts (xy 351.79 153.67) (xy 358.14 153.67))
     (stroke (width 0) (type default) (color 0 0 0 0))
@@
     (stroke (width 0) (type default) (color 0 0 0 0))
   )
+  (wire (pts (xy 25.4 55.88) (xy 27.94 55.88))
+    (stroke (width 0) (type default) (color 0 0 0 0))
+  )
   (wire (pts (xy 184.15 135.89) (xy 191.77 135.89))
     (stroke (width 0) (type default) (color 0 0 0 0))
@@
     (stroke (width 0) (type default) (color 0 0 0 0))
   )
+  (wire (pts (xy 69.85 58.42) (xy 69.85 57.15))
+    (stroke (width 0) (type default) (color 0 0 0 0))
+  )
   (wire (pts (xy 171.45 73.66) (xy 171.45 76.2))
+    (stroke (width 0) (type default) (color 0 0 0 0))
+  )
+  (wire (pts (xy 80.01 58.42) (xy 82.55 58.42))
     (stroke (width 0) (type default) (color 0 0 0 0))
   )
@@
     )
     (pin "1")
+  )
+  (symbol (lib_id "Device:C") (at 76.2 58.42 90) (unit 1)
+    (in_bom yes) (on_board yes)
+    (property "Reference" "C5" (id 0) (at 77.4701 60.96 0)
+      (effects (font (size 1.27 1.27)) (justify right))
+    )
+    (property "Value" "10uF" (id 1) (at 73.6601 59.69 0)
+      (effects (font (size 1.27 1.27)) (justify right))
+    )
+    (property "Footprint" "Capacitor_SMD:C_0805_2012Metric_Pad1.18x1.45mm_HandSolder" (id 2) (at 80.01 57.4548 0)
+      (effects (font (size 1.27 1.27)) hide)
+    )
+    (property "Datasheet" "~" (id 3) (at 76.2 58.42 0)
+      (effects (font (size 1.27 1.27)) hide)
+    )
+    (pin "1")
+    (pin "2")
   )
   (symbol (lib_id "Device:R_Small") (at 62.23 113.03 90) (unit 1)
@@
     (pin "2")
   )
+  (symbol (lib_id "Device:C") (at 31.75 55.88 90) (unit 1)
+    (in_bom yes) (on_board yes)
+    (property "Reference" "C4" (id 0) (at 33.0201 58.42 0)
+      (effects (font (size 1.27 1.27)) (justify right))
+    )
+    (property "Value" "10uF" (id 1) (at 29.2101 57.15 0)
+      (effects (font (size 1.27 1.27)) (justify right))
+    )
+    (property "Footprint" "Capacitor_SMD:C_0805_2012Metric_Pad1.18x1.45mm_HandSolder" (id 2) (at 35.56 54.9148 0)
+      (effects (font (size 1.27 1.27)) hide)
+    )
+    (property "Datasheet" "~" (id 3) (at 31.75 55.88 0)
+      (effects (font (size 1.27 1.27)) hide)
+    )
+    (pin "1")
+    (pin "2")
+  )
   (symbol (lib_id "Transistor_BJT:BC817") (at 60.96 214.63 0) (unit 1)
     (in_bom yes) (on_board yes) (fields_autoplaced)
@@
     (pin "2")
   )
+  (symbol (lib_id "power:GNDREF") (at 25.4 55.88 270) (unit 1)
+    (in_bom yes) (on_board yes)
+    (property "Reference" "#PWR0146" (id 0) (at 19.05 55.88 0)
+      (effects (font (size 1.27 1.27)) hide)
+    )
+    (property "Value" "GNDREF" (id 1) (at 15.24 55.8799 90)
+      (effects (font (size 1.27 1.27)) (justify left))
+    )
+    (property "Footprint" "" (id 2) (at 25.4 55.88 0)
+      (effects (font (size 1.27 1.27)) hide)
+    )
+    (property "Datasheet" "" (id 3) (at 25.4 55.88 0)
+      (effects (font (size 1.27 1.27)) hide)
+    )
+    (pin "1")
+  )
   (symbol (lib_id "power:GNDREF") (at 171.45 43.18 0) (unit 1)
     (in_bom yes) (on_board yes)
@@
     (pin "1")
   )
+  (symbol (lib_id "power:GNDREF") (at 82.55 58.42 90) (unit 1)
+    (in_bom yes) (on_board yes)
+    (property "Reference" "#PWR0145" (id 0) (at 88.9 58.42 0)
+      (effects (font (size 1.27 1.27)) hide)
+    )
+    (property "Value" "GNDREF" (id 1) (at 92.71 58.4201 90)
+      (effects (font (size 1.27 1.27)) (justify left))
+    )
+    (property "Footprint" "" (id 2) (at 82.55 58.42 0)
+      (effects (font (size 1.27 1.27)) hide)
+    )
+    (property "Datasheet" "" (id 3) (at 82.55 58.42 0)
+      (effects (font (size 1.27 1.27)) hide)
+    )
+    (pin "1")
+  )
   (symbol (lib_id "power:GNDREF") (at 78.74 49.53 90) (unit 1)
     (in_bom yes) (on_board yes)
@@
       (reference "#PWR0144") (unit 1) (value "GNDREF") (footprint "")
     )
+    (path "/e986394b-d7ab-4802-8e16-edc3ba842daf"
+      (reference "#PWR0145") (unit 1) (value "GNDREF") (footprint "")
+    )
+    (path "/cbe6df12-529c-4b15-851d-fb7ff22b8047"
+      (reference "#PWR0146") (unit 1) (value "GNDREF") (footprint "")
+    )
     (path "/80749d5f-f4c9-4f60-a934-338f9cb8414c"
       (reference "BT1") (unit 1) (value "Battery_pack") (footprint "GustavsGlobalLibrary:3xAA holder (534-2464)")
@@
       (reference "C3") (unit 1) (value "0.1uF") (footprint "Capacitor_SMD:C_0805_2012Metric_Pad1.18x1.45mm_HandSolder")
     )
+    (path "/69991fa4-5ce3-4154-b2cd-6875f56d0c77"
+      (reference "C4") (unit 1) (value "10uF") (footprint "Capacitor_SMD:C_0805_2012Metric_Pad1.18x1.45mm_HandSolder")
+    )
+    (path "/12244225-40cf-4940-a1fb-ce4acf762ae2"
+      (reference "C5") (unit 1) (value "10uF") (footprint "Capacitor_SMD:C_0805_2012Metric_Pad1.18x1.45mm_HandSolder")
+    )
     (path "/aefdd1a2-a196-4897-bd09-f4bc999af975"
